File: DC-Supply-170V-v1.kicad_pcb (KiCad board)
At the start: 2 copper layers, 94 x 78.7 mm, 47 parts, among them Q1 TIP50G, Q2 BSP16T1G, Q3 AO3162, Q4 AO3162, U1 LR8K4-G

Commit message: Layout tweaks before PCB order
Parts:
- moved D7 6.29 mm to (144.7, 58.4)
- moved C2 3.81 mm to (144.7, 63.0)
- moved D4 3.81 mm to (157.0, 63.0)
- moved Q4 3.81 mm to (157.0, 67.6)
- moved R6 3.81 mm to (151.9, 58.4)
- moved R7 3.81 mm to (144.8, 67.1)
- moved R8 3.81 mm to (157.0, 58.4)
- moved R9 3.81 mm to (154.2, 73.0)
- moved D3 3.81 mm to (151.8, 63.0)
- moved Q3 3.81 mm to (151.8, 67.6)
Routing:
- net LINE+: track 65.8 -> 72.0 mm
- net Net-(C2-Pad2): track 15.4 -> 13.0 mm
- net Vrect: track 155.3 -> 154.7 mm

Commit message: finalized before PCB order
Routing:
- net Net-(Q1-Pad2): track 46.8 -> 41.3 mm
- added copper zone on F.Cu, net Net-(Q1-Pad2)
Changed lines of the file:
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@@
     (thickness 1.6)
     (drawings 18)
-    (tracks 172)
+    (tracks 171)
     (zones 0)
     (modules 47)
@@
   (layers
     (0 F.Cu signal)
-    (31 B.Cu signal)
+    (31 B.Cu signal hide)
     (32 B.Adhes user hide)
     (33 F.Adhes user hide)
@@
     (add_net "Net-(R3-Pad1)")
   )
+  (module "Rays Footprints:TO-220-3_Horizontal_Tab4" (layer F.Cu)
+    (at 133.2738 95.6818 270)
+    (descr "TO-220-3, Horizontal, RM 2.54mm")
+    (tags "TO-220-3 Horizontal RM 2.54mm")
+    (fp_text reference Q1 (at -3.9878 -16.5862 180) (layer F.SilkS)
+      (effects (font (size 1.27 1.27) (thickness 0.2032)))
+    )
+    (fp_text value TIP50G (at 2.54 1.9 270) (layer F.Fab)
+      (effects (font (size 1 1) (thickness 0.15)))
+    )
+    (fp_circle (center 2.54 -16.66) (end 4.39 -16.66) (layer F.Fab) (width 0.1))
+    (fp_line (start 8.001 -19.939) (end -2.921 -19.939) (layer F.CrtYd) (width 0.05))
+    (fp_line (start 8.001 1.143) (end 8.001 -19.939) (layer F.CrtYd) (width 0.05))
+    (fp_line (start -2.921 1.143) (end 8.001 1.143) (layer F.CrtYd) (width 0.05))
+    (fp_line (start -2.921 -19.939) (end -2.921 1.143) (layer F.CrtYd) (width 0.05))
+    (fp_line (start 5.08 -3.69) (end 5.08 -1.066) (layer F.SilkS) (width 0.12))
+    (fp_line (start 2.54 -3.69) (end 2.54 -1.066) (layer F.SilkS) (width 0.12))
+    (fp_line (start 0 -3.69) (end 0 -1.05) (layer F.SilkS) (width 0.12))
+    (fp_line (start 7.874 -19.812) (end 7.874 -3.683) (layer F.SilkS) (width 0.12))
+    (fp_line (start -2.794 -19.812) (end -2.794 -3.683) (layer F.SilkS) (width 0.12))
+    (fp_line (start -2.794 -19.812) (end 7.874 -19.812) (layer F.SilkS) (width 0.12))
+    (fp_line (start -2.794 -3.683) (end 7.874 -3.683) (layer F.SilkS) (width 0.12))
+    (fp_line (start 5.08 -3.81) (end 5.08 0) (layer F.Fab) (width 0.1))
+    (fp_line (start 2.54 -3.81) (end 2.54 0) (layer F.Fab) (width 0.1))
+    (fp_line (start 0 -3.81) (end 0 0) (layer F.Fab) (width 0.1))
+    (fp_line (start 7.54 -3.81) (end -2.46 -3.81) (layer F.Fab) (width 0.1))
+    (fp_line (start 7.54 -13.06) (end 7.54 -3.81) (layer F.Fab) (width 0.1))
+    (fp_line (start -2.46 -13.06) (end 7.54 -13.06) (layer F.Fab) (width 0.1))
+    (fp_line (start -2.46 -3.81) (end -2.46 -13.06) (layer F.Fab) (width 0.1))
+    (fp_line (start 7.54 -13.06) (end -2.46 -13.06) (layer F.Fab) (width 0.1))
+    (fp_line (start 7.54 -19.46) (end 7.54 -13.06) (layer F.Fab) (width 0.1))
+    (fp_line (start -2.46 -19.46) (end 7.54 -19.46) (layer F.Fab) (width 0.1))
+    (fp_line (start -2.46 -13.06) (end -2.46 -19.46) (layer F.Fab) (width 0.1))
+    (fp_text user %R (at 2.54 -20.58 270) (layer F.Fab)
+      (effects (font (size 1 1) (thickness 0.15)))
+    )
+    (pad 3 thru_hole oval (at 5.08 0 270) (size 1.8 1.8) (drill 1) (layers *.Cu *.Mask)
+      (net 3 "Net-(Q1-Pad3)"))
+    (pad 2 thru_hole oval (at 2.54 0 270) (size 1.8 1.8) (drill 1) (layers *.Cu *.Mask)
+      (net 10 "Net-(Q1-Pad2)"))
+    (pad 1 thru_hole rect (at 0 0 270) (size 1.8 1.8) (drill 1) (layers *.Cu *.Mask)
+      (net 6 "Net-(Q1-Pad1)"))
+    (pad "" np_thru_hole oval (at 2.54 -16.66 270) (size 5.08 5.08) (drill 3.556) (layers *.Cu *.Mask))
+    (model ${KICAD_USER_LIB_DIR}/TO_SOT_Packages_THT.3dshapes/TO-220-3_Horizontal.wrl
+      (offset (xyz 2.539999961853027 0 0))
+      (scale (xyz 0.393701 0.393701 0.393701))
+      (rotate (xyz 0 0 0))
+    )
+    (model C:/Users/ray/OneDrive/Projects/kicad/3-3DModels/TO-220-3_Horizontal_TabDown.step
+      (at (xyz 0 0 0))
+      (scale (xyz 1 1 1))
+      (rotate (xyz 0 0 0))
+    )
+  )
   (module Connector_PinHeader_2.54mm:PinHeader_1x02_P2.54mm_Vertical (layer F.Cu)
     (at 163.322 77.2922)
@@
       (net 11 "Net-(Q2-Pad1)"))
     (model ${KISYS3DMOD}/Package_TO_SOT_SMD.3dshapes/SOT-223.wrl
-      (at (xyz 0 0 0))
-      (scale (xyz 1 1 1))
-      (rotate (xyz 0 0 0))
-    )
-  )
-  (module "Rays Footprints:TO-220-3_Horizontal_Tab4" (layer F.Cu)
-    (at 133.2738 95.6818 270)
-    (descr "TO-220-3, Horizontal, RM 2.54mm")
-    (tags "TO-220-3 Horizontal RM 2.54mm")
-    (fp_text reference Q1 (at -3.9878 -16.5862 180) (layer F.SilkS)
-      (effects (font (size 1.27 1.27) (thickness 0.2032)))
-    )
-    (fp_text value TIP50G (at 2.54 1.9 90) (layer F.Fab)
-      (effects (font (size 1 1) (thickness 0.15)))
-    )
-    (fp_circle (center 2.54 -16.66) (end 4.39 -16.66) (layer F.Fab) (width 0.1))
-    (fp_line (start 8.001 -19.939) (end -2.921 -19.939) (layer F.CrtYd) (width 0.05))
-    (fp_line (start 8.001 1.143) (end 8.001 -19.939) (layer F.CrtYd) (width 0.05))
-    (fp_line (start -2.921 1.143) (end 8.001 1.143) (layer F.CrtYd) (width 0.05))
-    (fp_line (start -2.921 -19.939) (end -2.921 1.143) (layer F.CrtYd) (width 0.05))
-    (fp_line (start 5.08 -3.69) (end 5.08 -1.066) (layer F.SilkS) (width 0.12))
-    (fp_line (start 2.54 -3.69) (end 2.54 -1.066) (layer F.SilkS) (width 0.12))
-    (fp_line (start 0 -3.69) (end 0 -1.05) (layer F.SilkS) (width 0.12))
-    (fp_line (start 7.874 -19.812) (end 7.874 -3.683) (layer F.SilkS) (width 0.12))
-    (fp_line (start -2.794 -19.812) (end -2.794 -3.683) (layer F.SilkS) (width 0.12))
-    (fp_line (start -2.794 -19.812) (end 7.874 -19.812) (layer F.SilkS) (width 0.12))
-    (fp_line (start -2.794 -3.683) (end 7.874 -3.683) (layer F.SilkS) (width 0.12))
-    (fp_line (start 5.08 -3.81) (end 5.08 0) (layer F.Fab) (width 0.1))
-    (fp_line (start 2.54 -3.81) (end 2.54 0) (layer F.Fab) (width 0.1))
-    (fp_line (start 0 -3.81) (end 0 0) (layer F.Fab) (width 0.1))
-    (fp_line (start 7.54 -3.81) (end -2.46 -3.81) (layer F.Fab) (width 0.1))
-    (fp_line (start 7.54 -13.06) (end 7.54 -3.81) (layer F.Fab) (width 0.1))
-    (fp_line (start -2.46 -13.06) (end 7.54 -13.06) (layer F.Fab) (width 0.1))
-    (fp_line (start -2.46 -3.81) (end -2.46 -13.06) (layer F.Fab) (width 0.1))
-    (fp_line (start 7.54 -13.06) (end -2.46 -13.06) (layer F.Fab) (width 0.1))
-    (fp_line (start 7.54 -19.46) (end 7.54 -13.06) (layer F.Fab) (width 0.1))
-    (fp_line (start -2.46 -19.46) (end 7.54 -19.46) (layer F.Fab) (width 0.1))
-    (fp_line (start -2.46 -13.06) (end -2.46 -19.46) (layer F.Fab) (width 0.1))
-    (fp_text user %R (at 2.54 -20.58 90) (layer F.Fab)
-      (effects (font (size 1 1) (thickness 0.15)))
-    )
-    (pad 3 thru_hole oval (at 5.08 0 270) (size 1.8 1.8) (drill 1) (layers *.Cu *.Mask)
-      (net 3 "Net-(Q1-Pad3)"))
-    (pad 2 thru_hole oval (at 2.54 0 270) (size 1.8 1.8) (drill 1) (layers *.Cu *.Mask)
-      (net 10 "Net-(Q1-Pad2)"))
-    (pad 1 thru_hole rect (at 0 0 270) (size 1.8 1.8) (drill 1) (layers *.Cu *.Mask)
-      (net 6 "Net-(Q1-Pad1)"))
-    (pad 4 np_thru_hole oval (at 2.54 -16.66 270) (size 3.5 3.5) (drill 3.5) (layers *.Cu *.Mask)
-      (net 10 "Net-(Q1-Pad2)"))
-    (model ${KICAD_USER_LIB_DIR}/TO_SOT_Packages_THT.3dshapes/TO-220-3_Horizontal.wrl
-      (offset (xyz 2.539999961853027 0 0))
-      (scale (xyz 0.393701 0.393701 0.393701))
-      (rotate (xyz 0 0 0))
-    )
-    (model C:/Users/ray/OneDrive/Projects/kicad/3-3DModels/TO-220-3_Horizontal_TabDown.step
       (at (xyz 0 0 0))
       (scale (xyz 1 1 1))
@@
   (segment (start 110.414 102.489) (end 103.378 102.489) (width 1.651) (layer F.Cu) (net 8) (status 30))
   (segment (start 110.395 108.585) (end 103.378 108.585) (width 1.651) (layer F.Cu) (net 9) (status 30))
-  (segment (start 133.2484 98.1964) (end 138.7856 98.1964) (width 1.778) (layer F.Cu) (net 10) (status 10))
-  (segment (start 138.811 98.2218) (end 149.9338 98.2218) (width 1.778) (layer F.Cu) (net 10) (status 20))
   (segment (start 138.7856 98.1964) (end 138.811 98.2218) (width 0.762) (layer F.Cu) (net 10))
   (segment (start 161.036 86.995) (end 161.036 90.805) (width 1.778) (layer F.Cu) (net 10) (status 30))
@@
   (segment (start 138.7856 98.1964) (end 148.463 88.519) (width 1.778) (layer F.Cu) (net 10))
   (segment (start 148.463 88.519) (end 160.909 88.519) (width 1.778) (layer F.Cu) (net 10))
+  (segment (start 133.2484 98.1964) (end 144.399 98.1964) (width 1.778) (layer F.Cu) (net 10))
   (segment (start 123.2522 99.575) (end 123.2408 99.5864) (width 0.762) (layer F.Cu) (net 11) (status 30))
   (segment (start 123.2522 96.0378) (end 123.2522 99.575) (width 0.762) (layer F.Cu) (net 11) (status 30))
@@
       )
     )
+  )
+  (zone (net 10) (net_name "Net-(Q1-Pad2)") (layer F.Cu) (hatch edge 0.508)
+    (connect_pads (clearance 0.254))
+    (min_thickness 0.254)
+    (fill yes (arc_segments 32) (thermal_gap 0.508) (thermal_bridge_width 0.508))
+    (polygon
+      (pts
+        (xy 153.797 104.267) (xy 136.906 104.267) (xy 136.906 92.202) (xy 153.797 92.202)
+      )
+    )
+  )
+  (zone (net 0) (net_name "") (layer F.Mask) (hatch edge 0.508)
+    (connect_pads (clearance 0.254))
+    (min_thickness 0.254)
+    (fill yes (arc_segments 32) (thermal_gap 0.508) (thermal_bridge_width 0.508))
+    (polygon
+      (pts
+        (xy 154.051 104.521) (xy 136.652 104.521) (xy 136.652 91.948) (xy 154.051 91.948)
+      )
+    )
